File: GA_Fuelstation_Terminal.kicad_pcb (KiCad board)
At the start: 2 copper layers, 136.6 x 58.4 mm, 36 parts, among them IC1 ESP32-S3-WROOM-1, J1 Conn_01x08_Pin, J10 Screw_Terminal_01x02, J2 Conn_01x05_Pin, J5 Conn_01x02_Pin, J6 Screw_Terminal_01x02, J7 Screw_Terminal_01x02, J98 Conn_01x07_Socket, J99 Conn_ARM_JTAG_SWD_20, Q1 2N7002, Q2 2N7002, Q3 2N7002, U1 3V3, U2 5V

Commit message: Adapted gitignore Add LAN Add USB2RS232
Parts:
- added C3: 1uF/16V, Capacitor_SMD:C_0603_1608Metric, F.Cu at (54.2, 48.3)
- added C4: 10uF/25V, Capacitor_SMD:C_0603_1608Metric, F.Cu at (54.2, 50.8)
- added D2: LESD5D5.0CT1G, Diode_SMD:D_SOD-523, F.Cu at (50.4, 48.3)
- added D3: LESD5D5.0CT1G, Diode_SMD:D_SOD-523, F.Cu at (50.4, 50.7)
- added D4: LESD5D5.0CT1G, Diode_SMD:D_SOD-523, F.Cu at (50.4, 53.2)
- added J3: USB_C_Receptacle_USB2.0_14P, Connector_USB:USB_C_Receptacle_HRO_TYPE-C-31-M-12, F.Cu at (43.7, 42.6)
- added J8: Screw_Terminal_01x02, Connector_Phoenix_MSTB:PhoenixContact_MSTBA_2,5_2-G-5,08_1x02_P5.08mm_Horizontal, F.Cu at (145.8, 119.7)
- added Q4: L8050QLT1G, Package_TO_SOT_SMD:SOT-23, F.Cu at (46.1, 49.3)
- added Q5: L8050QLT1G, Package_TO_SOT_SMD:SOT-23, F.Cu at (46.1, 53.7)
- added R11: R, Resistor_SMD:R_0603_1608Metric_Pad0.98x0.95mm_HandSolder, F.Cu at (87.6, 53.3)
- added R12: R, Resistor_SMD:R_0603_1608Metric_Pad0.98x0.95mm_HandSolder, F.Cu at (87.6, 55.9)
- added R13: 22k1, Resistor_SMD:R_0402_1005Metric, F.Cu at (39.3, 48.0)
- added R14: 47k5, Resistor_SMD:R_0402_1005Metric, F.Cu at (39.3, 50.0)
- added R15: 1k, Resistor_SMD:R_0402_1005Metric, F.Cu at (39.3, 52.0)
- added R16: 10K, Resistor_SMD:R_0402_1005Metric, F.Cu at (39.3, 54.0)
- added R17: 10K, Resistor_SMD:R_0402_1005Metric, F.Cu at (39.3, 56.0)
- added R18: 10K, Resistor_SMD:R_0402_1005Metric, F.Cu at (42.2, 48.0)
- added R19: 0R, Resistor_SMD:R_0402_1005Metric, F.Cu at (42.2, 50.0)
- added R20: 0R, Resistor_SMD:R_0402_1005Metric, F.Cu at (42.2, 52.0)
- added R21: 0R, Resistor_SMD:R_0402_1005Metric, F.Cu at (42.2, 54.0)
- added R22: 0R, Resistor_SMD:R_0402_1005Metric, F.Cu at (42.2, 56.0)
- added U3: EL817, Package_SO:SOP-4_3.8x4.1mm_P2.54mm, F.Cu at (142.2, 110.5)
- added U4: WIZ850io, GA_Fuelstation_Terminal:WIZ850io, F.Cu at (197.6, 126.2)
- added U5: CP2102N-Axx-xQFN28, Package_DFN_QFN:QFN-28-1EP_5x5mm_P0.5mm_EP3.35x3.35mm, F.Cu at (53.2, 41.2)
- C10: value 100nF / 50V -> 100nF / 50V
Connections:
- net MISO renamed RFID_MISO
- net MOSI renamed RFID_MOSI
- J1 pad 2: SCK -> RFID_SCK

Commit message: Add input protection, fix USB-C/CP2102 supply, harden optocoupler input
Power supply:
- Add 12V input protection: PTC fuse F1 (1.1A/33V, C70119), TVS D6
  (SMAJ15CA, C151939), reverse polarity Schottky D7 (SS34, C8678) and
  bulk cap C13 (100uF/25V, C179802)

USB2RS232:
- Power CP2102N (VDD/REGIN) from +3.3V via R25 (0R)
- Add 5k1 pull-downs R23/R24 on USB-C CC1/CC2 so C-to-C hosts supply VBUS

ESP32 / Interfaces:
- Add 100k gate pull-downs R26/R27/R28 on Q2/Q1/Q3 (relay, LED, buzzer
  stay off during reset/boot)
- Buzzer flyback D1: 1N4148W SOD-123 (C81598) instead of undefined SOT-23
- WAKE_UP input (J8/U3): series zener D8 (BZT52C6V8, C173404), reverse
  polarity diode D9 (1N4148W), R11 = 1k5 0805 (C4310); switches at ~9V,
  safe up to 14.4V
- IC1 value set to ESP32-S3-WROOM-1U to match footprint
- Add no-connect flags on unused ESP32, J99 and K1 pins
- Remove duplicate local labels IO_PUMP_LED/IO_PUMP_RELAIS
- Move off-grid symbols, labels and wires onto grid

PCB: update from schematic
Parts:
- added C13: 100uF/25V, Capacitor_SMD:CP_Elec_6.3x7.7, F.Cu at (161.4, 25.4)
- added D5: 1N4148W, Diode_SMD:D_SOD-123, F.Cu at (176.2, 23.0)
- added D6: SMAJ15CA, Diode_SMD:D_SMA, F.Cu at (160.3, 31.8)
- added D7: SS34, Diode_SMD:D_SMA, F.Cu at (160.3, 36.3)
- added F1: PTC 1.1A/30V, Fuse:Fuse_1812_4532Metric, F.Cu at (167.8, 32.0)
- added R23: 5k1, Resistor_SMD:R_0603_1608Metric_Pad0.98x0.95mm_HandSolder, F.Cu at (175.4, 31.9)
- added R24: 5k1, Resistor_SMD:R_0603_1608Metric_Pad0.98x0.95mm_HandSolder, F.Cu at (175.4, 34.4)
- added R25: 0R, Resistor_SMD:R_0402_1005Metric_Pad0.72x0.64mm_HandSolder, F.Cu at (174.9, 36.7)
- added R26: 100k, Resistor_SMD:R_0402_1005Metric_Pad0.72x0.64mm_HandSolder, F.Cu at (174.9, 25.7)
- added R27: 100k, Resistor_SMD:R_0402_1005Metric_Pad0.72x0.64mm_HandSolder, F.Cu at (174.9, 27.7)
- added R28: 100k, Resistor_SMD:R_0402_1005Metric_Pad0.72x0.64mm_HandSolder, F.Cu at (174.9, 40.7)
- D1: value D -> 1N4148W; footprint Package_TO_SOT_SMD:SOT-23 -> Diode_SMD:D_SOD-123
- R12: value R -> 10k
Connections:
- IC1 pad 20: SCK -> RFID_SCK
- IC1 pad 22: unconnected-(IC1-GPIO14/TOUCH14/ADC2_CH3/FSPIWP/FSPIDQS/SUBSPIWP-Pad22) -> LAN_SCK
- IC1 pad 23: unconnected-(IC1-GPIO21-Pad23) -> WAKE_UP
- IC1 pad 5: unconnected-(IC1-GPIO5/TOUCH5/ADC1_CH4-Pad5) -> LAN_CS
- IC1 pad 6: unconnected-(IC1-GPIO6/TOUCH6/ADC1_CH5-Pad6) -> LAN_RST
- IC1 pad 7: unconnected-(IC1-GPIO7/TOUCH7/ADC1_CH6-Pad7) -> LAN_INT
- IC1 pad 8: unconnected-(IC1-GPIO15/U0RTS/ADC2_CH4/XTAL_32K_P-Pad8) -> LAN_MISO
- IC1 pad 9: unconnected-(IC1-GPIO16/U0CTS/ADC2_CH5/XTAL_32K_N-Pad9) -> LAN_MOSI
- J10 pad 1: +12V -> Net-(J10-Pin_1)
- J3 pad A5: unconnected-(J3-CC1-PadA5) -> Net-(J3-CC1)
- J3 pad B5: unconnected-(J3-CC2-PadB5) -> Net-(J3-CC2)
- R12 pad 1: +3V3 -> +3.3V
- U4 pad 10: +3V3 -> +3.3V
- U4 pad 11: +3V3 -> +3.3V
Routing:
- net SCK: track 48.7 -> 0.00 mm
- net RFID_SCK: track 0.00 -> 48.7 mm

Commit message: - Q4/Q5: use MMBT3904 symbol (numbered pins) so SOT-23 pads map correctly
Parts:
- added D8: BZT52C6V8, Diode_SMD:D_SOD-123, F.Cu at (198.3, 29.1)
- added D9: 1N4148W, Diode_SMD:D_SOD-123, F.Cu at (198.3, 32.5)
- IC1: value ESP32-S3-WROOM-1 -> ESP32-S3-WROOM-1U
- R11: value R -> 1k5; footprint Resistor_SMD:R_0603_1608Metric_Pad0.98x0.95mm_HandSolder -> Resistor_SMD:R_0805_2012Metric_Pad1.20x1.40mm_HandSolder
Connections:
- J8 pad 2: Net-(J8-Pin_2) -> Net-(D8-K)
- Q4 pad 1: (no net) -> Net-(Q4-B)
- Q4 pad 2: (no net) -> /USB2RS232/CP2102_RTS
- Q4 pad 3: (no net) -> Net-(Q4-C)
- Q5 pad 1: (no net) -> Net-(Q5-B)
- Q5 pad 2: (no net) -> /USB2RS232/CP2102_DTR
- Q5 pad 3: (no net) -> Net-(Q5-C)
- R11 pad 1: Net-(J8-Pin_2) -> Net-(D8-A)
- R17 pad 2: Net-(Q5-PadB) -> Net-(Q5-B)
- R18 pad 2: Net-(Q4-PadB) -> Net-(Q4-B)
- R19 pad 1: Net-(Q5-PadC) -> Net-(Q5-C)
- R20 pad 1: Net-(Q4-PadC) -> Net-(Q4-C)

Commit message: Add native ESP32-S3 USB port, move buzzer driver to Interfaces sheet
ESP32:
- Add USB-C J4 for ESP32-S3 native USB (USB-Serial-JTAG):
  D+ -> GPIO20, D- -> GPIO19 via 0R series resistors R31/R32 (0402, C17168),
  ESD diodes D10/D12 (LESD5D5.0CT1G), CC pull-downs R29/R30 5k1,
  VBUS not connected (no-connect flag)
- Move JTAG header J99 and decoupling C10-C12 to free space for J4

Interfaces:
- Move buzzer driver (Q3, R6, R28, R2, R7, D1, BZ1) from ESP32 sheet
- Make IO_BUZZER a global label so GPIO4 still reaches R6/Q3
- Shift optocoupler input block (J8, D8, D9, R11, R12, U3) down

Power supply:
- Add PWR_FLAG on +12V after reverse polarity diode D7 (ERC clean)

PCB: update from schematic
ERC: 0 errors, 5 warnings (2N7002 symbol lib mismatch, unused RFID_IRQ/RST)
Parts:
- added D10: LESD5D5.0CT1G, Diode_SMD:D_SOD-523, F.Cu at (221.1, 36.6)
- added D12: LESD5D5.0CT1G, Diode_SMD:D_SOD-523, F.Cu at (221.1, 39.0)
- added J4: USB_C_Receptacle_USB2.0_14P, Connector_USB:USB_C_Receptacle_HRO_TYPE-C-31-M-12, F.Cu at (220.7, 30.7)
- added R29: 5k1, Resistor_SMD:R_0603_1608Metric_Pad0.98x0.95mm_HandSolder, F.Cu at (217.1, 36.6)
- added R30: 5k1, Resistor_SMD:R_0603_1608Metric_Pad0.98x0.95mm_HandSolder, F.Cu at (217.1, 39.1)
- added R31: 0R, Resistor_SMD:R_0402_1005Metric, F.Cu at (224.3, 36.4)
- added R32: 0R, Resistor_SMD:R_0402_1005Metric, F.Cu at (224.3, 38.4)
Connections:
- net /ESP32/IO_BUZZER renamed IO_BUZZER
- IC1 pad 13: unconnected-(IC1-GPIO19/U1RTS/ADC2_CH8/CLK_OUT2/USB_D--Pad13) -> /ESP32/DEBUG_USB_DN
- IC1 pad 14: unconnected-(IC1-GPIO20/U1CTS/ADC2_CH9/CLK_OUT1/USB_D+-Pad14) -> /ESP32/DEBUG_USB_DP
