File: esp32.kicad_sch (KiCad schematic)
At the start: 14 parts, among them IC1 ESP32-S3-WROOM-1, J10 Conn_01x07_Socket, J99 Conn_ARM_JTAG_SWD_20, Q3 2N7002

Commit message: LAN PHy
Parts:
- removed IC1: ESP32-S3-WROOM-1, Espressif:ESP32-S3-WROOM-1U, symbol Espressif:ESP32-S3-WROOM-1
- removed J99: Conn_ARM_JTAG_SWD_20, Connector_IDC:IDC-Header_2x10_P2.54mm_Vertical, symbol Connector:Conn_ARM_JTAG_SWD_20
- added U3: ESP32-WROVER-E, Espressif:ESP32-WROVER-E, symbol Espressif:ESP32-WROVER-E
- C1: value 1u -> 4u7
- C10: value 100nF / 50V -> 100nF / 50V
- D1: value D -> 1N4148; footprint Package_TO_SOT_SMD:SOT-23 -> Diode_SMD:D_SOD-323_HandSoldering
- R7: renamed from R6; value R -> 0R
- renumbered J10 to J98, R7 to R6
Connections:
- net +3.3V: now also U3.2 (3V3)
- net EN: now also U3.3 (EN/CHIP_PU)
- net GND: now also U3.1 (GND), U3.15 (GND), U3.38 (GND), U3.39 (GND_THERMAL)
- net IO0: now also U3.25 (GPIO0/BOOT/ADC2_CH1)
- net IO_BUZZER: now also U3.26 (ADC2_CH0/GPIO4)
- net IO_PUMP_LED: now also U3.24 (ADC2_CH2/GPIO2)
- net IO_PUMP_PULSE: now also U3.6 (GPIO34/ADC1_CH6)
- net IO_PUMP_RELAIS: now also U3.29 (GPIO5)
- net RFID_SS: now also U3.23 (MTDO/GPIO15/ADC2_CH3)
- net RXD: now also U3.35 (U0TXD/GPIO1)
- net SCK: now also U3.13 (MTMS/GPIO14/ADC2_CH6)
- net SCL: now also U3.8 (32K_XP/GPIO32/ADC1_CH4)
- net SDA: now also U3.9 (32K_XN/GPIO33/ADC1_CH5)
- net TXD: now also U3.34 (U0RXD/GPIO3)
- new net EMAC_CRS_DV: U3.12 (ADC2_CH7/GPIO27)
- new net EMAC_RXD0: U3.10 (DAC_1/ADC2_CH8/GPIO25)
- new net EMAC_RXD1: U3.11 (DAC_2/ADC2_CH9/GPIO26)
- new net EMAC_TXD0: U3.31 (GPIO19)
- new net EMAC_TXD1: U3.36 (GPIO22)
- new net EMAC_TX_EN: U3.33 (GPIO21)
- new net MDC: U3.37 (GPIO23)
- new net MDIO: U3.30 (GPIO18)
- new net WAKEUP: U3.4 (SENSOR_VP/GPIO36/ADC1_CH0)
Other:
- note added: "Add Reset Taster"
- moved on the sheet: C1, D1, R1
