File: interfaces.kicad_sch (KiCad schematic)
At the start: 19 parts, among them J2 Screw_Terminal_01x02, J4 Conn_01x05_Pin, J5 Conn_01x08_Pin, J6 Conn_01x02_Pin, Q1 2N7002, Q2 2N7002

Commit message: LAN PHy
Parts:
- added J3: Screw_Terminal_01x02, Connector_Phoenix_MSTB:PhoenixContact_MSTBA_2,5_2-G-5,08_1x02_P5.08mm_Horizontal, symbol Connector:Screw_Terminal_01x02
- added R11, R12: R, Resistor_SMD:R_0402_1005Metric_Pad0.72x0.64mm_HandSolder, symbol Device:R
- added U4: EL817, Package_DIP:SMDIP-4_W7.62mm, symbol Isolator:EL817
- K1: value ~ -> (none)
- R9: value 50k -> 68k
- renumbered J5 to J1, J4 to J2, J6 to J5, J2 to J6, J2 to J7
Connections:
- net GND: now also U4.3
- net IO_PUMP_PULSE: now also R9.2
- net at J7.1 (Pin_1), R8.2: no longer R9.2
- new net: J3.1 (Pin_1), R11.1
- new net: J3.2 (Pin_2), U4.2
- new net: R11.2, U4.1
- new net +3V3: R12.1
- new net WAKEUP: R12.2, U4.4
Other:
- moved on the sheet: R9
